Commit message: Added launch file for controlling the arm positions without using moveit

File: simulation/grasping_sim/urdf/urdf/common.xacro (robot description, xacro)
@@ -43,5 +43,5 @@
         <hardwareInterface>PositionJointInterface</hardwareInterface>
         <hardwareInterface>VelocityJointInterface</hardwareInterface>
-        <!--hardwareInterface>EffortJointInterface</hardwareInterface-->
+        <hardwareInterface>EffortJointInterface</hardwareInterface>
       </joint>
       <actuator name="${jname}_motor">

File: simulation/grasping_sim/urdf/urdf/lwa4p/lwa4p.gazebo.xacro (robot description, xacro)
@@ -5,35 +5,35 @@
       <gravity>true</gravity>
       <self_collide>false</self_collide>
-      <material value="Schunk/LightGrey" />
+      <material value="Gazebo/LightGrey" />
     </gazebo>
     <gazebo reference="${name}_1_link">
       <gravity>true</gravity>
       <self_collide>false</self_collide>
-      <material value="Schunk/Blue" />
+      <material value="Gazebo/Blue" />
     </gazebo>
     <gazebo reference="${name}_2_link">
       <gravity>true</gravity>
       <self_collide>false</self_collide>
-      <material value="Schunk/LightGrey" />
+      <material value="Gazebo/LightGrey" />
     </gazebo>
     <gazebo reference="${name}_3_link">
       <gravity>true</gravity>
       <self_collide>false</self_collide>
-      <material value="Schunk/Blue" />
+      <material value="Gazebo/Blue" />
     </gazebo>
     <gazebo reference="${name}_4_link">
       <gravity>true</gravity>
       <self_collide>false</self_collide>
-      <material value="Schunk/LightGrey" />
+      <material value="Gazebo/LightGrey" />
     </gazebo>
     <gazebo reference="${name}_5_link">
       <gravity>true</gravity>
       <self_collide>false</self_collide>
-      <material value="Schunk/Blue" />
+      <material value="Gazebo/Blue" />
     </gazebo>
     <gazebo reference="${name}_6_link">
       <gravity>true</gravity>
       <self_collide>false</self_collide>
-      <material value="Schunk/LightGrey" />
+      <material value="Gazebo/LightGrey" />
     </gazebo>
   </xacro:macro>
