Commit message: Added files for hand simulation

File: simulation/grasping_sim/urdf/urdf/lwa4p/lwa4p.urdf.xacro (robot description, xacro)
@@ -2,5 +2,5 @@
 <robot xmlns:xacro="http://www.ros.org/wiki/xacro">
   <xacro:property name="safety_offset" value="0.02"/>
-  <xacro:include filename="$(find grasping_sim)/urdf/urdf/common.xacro" />
+  <xacro:include filename="$(find grasping_sim)/urdf/urdf/common.xacro"/>
   <xacro:include filename="$(find grasping_sim)/urdf/urdf/lwa4p/lwa4p.gazebo.xacro" />
   <xacro:include filename="$(find grasping_sim)/urdf/urdf/lwa4p/lwa4p.transmission.xacro" />

File: simulation/grasping_sim/urdf/urdf/svh/svh.urdf.xacro (robot description, xacro)
@@ -1,581 +1,598 @@
 <?xml version="1.0"?>
 <robot xmlns:xacro="http://www.ros.org/wiki/xacro">
-  <xacro:property name="cyl_radius" value="0.001" />
-  <xacro:macro name="svh" params="parent name side *origin">
-    <!-- RIGHT HAND = 1, LEFT HAND = -1 -->
-    <!-- BASE_LINE LINKS -->
-    <joint name="${name}_base_joint" type="fixed" >
-      <xacro:insert_block name="origin" />
-      <parent link="${parent}" />
-      <child link="${name}_base_link" />
-    </joint>
-    <link name="${name}_base_link">
-      <xacro:insert_block name="origin" />
-      <visual>
-	<origin xyz="0 0 -0.032" rpy="0 0 0" />
-	<geometry>
-          <mesh filename="package://schunk_lwa4p_svh/description/meshes/svh/base10.dae" />
-	</geometry>
-      </visual>
-      <collision>
-	<origin xyz="0 0 -0.032" rpy="0 0 0" />
-	<geometry>
-          <mesh filename="package://schunk_lwa4p_svh/description/meshes/svh/base10.dae" />
-	</geometry>
-      </collision>
-    </link>
-    <link name="${name}_d">
-      <!-- <visual> -->
-      <!-- 	<geometry> -->
-      <!-- 	  <cylinder length="0.110" radius="${cyl_radius}" /> -->
-      <!-- 	</geometry> -->
-      <!-- 	<material name="${name}_green" /> -->
-      <!-- </visual> -->
-    </link>
-    <link name="${name}_h">
-      <!-- <visual> -->
-      <!-- 	<origin rpy="0 1.571 0" xyz="${side*(-0.0125)} 0 0.0825" /> -->
-      <!-- 	<geometry> -->
-      <!-- 	  <cylinder length="0.025" radius="${cyl_radius}" /> -->
-      <!-- 	</geometry> -->
-      <!-- 	<material name="${name}_green" /> -->
-      <!-- </visual> -->
-    </link>
-    <link name="${name}_d2">
-      <!-- <visual> -->
-      <!-- 	<origin rpy="0 0 0" xyz="${side*(-0.025)} 0 0.09625" /> -->
-      <!-- 	<geometry> -->
-      <!-- 	  <cylinder length="0.0275" radius="${cyl_radius}" /> -->
-      <!-- 	</geometry> -->
-      <!-- 	<material name="${name}_green" /> -->
-      <!-- </visual> -->
-    </link>
-    <!-- LENGTH NOT FOUND IN DATASHEET! GUESSED!!! -->
-    <link name="${name}_e1">
-      <visual>
-	<origin rpy="0 0 0" xyz="0 0.01313 0" />
-	<geometry>
-          <mesh scale="${side*(1)} 1 1" filename="package://schunk_lwa4p_svh/description/meshes/svh/h10.dae" />
-	</geometry>
-      </visual>
-      <collision>
-	<origin rpy="0 0 0" xyz="0 0.01313 0" />
-	<geometry>
-          <mesh scale="${side*(1)} 1 1" filename="package://schunk_lwa4p_svh/description/meshes/svh/h10.dae" />
-	</geometry>
-      </collision>
-    </link>
-    <!-- LENGTH NOT FOUND IN DATASHEET! GUESSED!!! -->
-    <link name="${name}_e2">
-      <visual>
-	<origin xyz="${side*(-0.0007)} 0 -0.01002" />
-	<geometry>
-          <mesh scale="${side*(1)} 1 1" filename="package://schunk_lwa4p_svh/description/meshes/svh/h11.dae" />
-	</geometry>
-      </visual>
-      <collision>
-	<origin xyz="${side*(-0.0007)} 0 -0.01002" />
-	<geometry>
-          <mesh scale="${side*(1)} 1 1" filename="package://schunk_lwa4p_svh/description/meshes/svh/h11.dae" />
-	</geometry>
-      </collision>
-    </link>
-    <!-- LENGTH NOT FOUND IN DATASHEET! GUESSED!!! -->
-    <link name="${name}_e3">
-      <!-- <visual> -->
-      <!-- 	<origin rpy="0 0 0" xyz="${side*(0.0175)} 0 0.015" /> -->
-      <!-- 	<geometry> -->
-      <!-- 	  <cylinder length="0.03" radius="${cyl_radius}" /> -->
-      <!-- 	</geometry> -->
-      <!-- 	<material name="green" /> -->
-      <!-- </visual> -->
-    </link>
-    <link name="${name}_e">
-    </link>
-    <!-- LENGTH NOT FOUND IN DATASHEET! GUESSED, BUT POSITION CALCULATED: E4 = D-G-F!!! -->
-    <link name="${name}_e4">
-      <!-- <visual> -->
-      <!-- 	<origin rpy="0 0 0" xyz="${side*(0.02825)} 0 0.043" /> -->
-      <!-- 	<geometry> -->
-      <!-- 	  <cylinder length="0.026" radius="${cyl_radius}" /> -->
-      <!-- 	</geometry> -->
-      <!-- 	<material name="green" /> -->
-      <!-- </visual> -->
-    </link>
-    <!-- LENGTH NOT FOUND IN DATASHEET! GUESSED, BUT POSITION CALCULATED: E5 = D-G!!! -->
-    <link name="${name}_e5">
-      <!-- <visual> -->
-      <!-- 	<origin rpy="0 0 0" xyz="${side*(0.00675)} 0 0.04775" /> -->
-      <!-- 	<geometry> -->
-      <!-- 	  <cylinder length="0.0355" radius="${cyl_radius}" /> -->
-      <!-- 	</geometry> -->
-      <!-- 	<material name="green" /> -->
-      <!-- </visual> -->
-    </link>
-    <!-- THUMB LINKS -->
-    <link name="${name}_z">
-      <visual>
-	<origin xyz="0 0 0.02442" />
-	<geometry>
-          <mesh scale="1 ${side*(1)} 1" filename="package://schunk_lwa4p_svh/description/meshes/svh/d10.dae" />
-	</geometry>
-      </visual>
-      <collision>
-	<origin xyz="0 0 0.02442" />
-	<geometry>
-          <mesh scale="1 ${side*(1)} 1" filename="package://schunk_lwa4p_svh/description/meshes/svh/d10.dae" />
-	</geometry>
-      </collision>
-    </link>
-    <link name="${name}_virtual_a" />
-    <link name="${name}_a">
-      <visual>
-	<geometry>
-          <mesh scale="1 ${side*(1)} ${side*(1)}" filename="package://schunk_lwa4p_svh/description/meshes/svh/d11.dae" />
-	</geometry>
-      </visual>
-      <collision>
-	<geometry>
-          <mesh scale="1 ${side*(1)} ${side*(1)}" filename="package://schunk_lwa4p_svh/description/meshes/svh/d11.dae" />
-	</geometry>
-      </collision>
-    </link>
-    <link name="${name}_b">
-      <visual>
-	<geometry>
-          <mesh scale="1 ${side*(1)} ${side*(1)}" filename="package://schunk_lwa4p_svh/description/meshes/svh/d12.dae" />
-	</geometry>
-      </visual>
-      <collision>
-	<geometry>
-          <mesh scale="1 ${side*(1)} ${side*(1)}" filename="package://schunk_lwa4p_svh/description/meshes/svh/d12.dae" />
-	</geometry>
-      </collision>
-    </link>
-    <link name="${name}_c">
-      <visual>
-	<geometry>
-          <mesh scale="1 ${side*(1)} ${side*(1)}" filename="package://schunk_lwa4p_svh/description/meshes/svh/d13.dae" />
-	</geometry>
-      </visual>
-      <collision>
-	<geometry>
-          <mesh scale="1 ${side*(1)} ${side*(1)}" filename="package://schunk_lwa4p_svh/description/meshes/svh/d13.dae" />
-	</geometry>
-      </collision>
-    </link>
-    <!-- INDEX FINGER LINKS -->
-    <link name="${name}_virtual_l">
-      <visual>
-	<origin xyz="0 0 0.01321" />
-	<geometry>
-          <mesh filename="package://schunk_lwa4p_svh/description/meshes/svh/f10.dae" />
-	</geometry>
-      </visual>
-      <collision>
-	<origin xyz="0 0 0.01321" />
-	<geometry>
-          <mesh filename="package://schunk_lwa4p_svh/description/meshes/svh/f10.dae" />
-	</geometry>
-      </collision>
-    </link>
-    <link name="${name}_l">
-      <visual>
-	<geometry>
-          <mesh filename="package://schunk_lwa4p_svh/description/meshes/svh/f11.dae" />
-	</geometry>
-      </visual>
-      <collision>
-	<geometry>
-          <mesh filename="package://schunk_lwa4p_svh/description/meshes/svh/f11.dae" />
-	</geometry>
-      </collision>
-    </link>
-    <link name="${name}_p">
-      <visual>
-	<geometry>
-          <mesh filename="package://schunk_lwa4p_svh/description/meshes/svh/f12.dae" />
-	</geometry>
-      </visual>
-      <collision>
-	<geometry>
-          <mesh filename="package://schunk_lwa4p_svh/description/meshes/svh/f12.dae" />
-	</geometry>
-      </collision>
-    </link>
-    <link name="${name}_t">
-      <visual>
-	<geometry>
-          <mesh filename="package://schunk_lwa4p_svh/description/meshes/svh/f13.dae" />
-	</geometry>
-      </visual>
-      <collision>
-	<geometry>
-          <mesh filename="package://schunk_lwa4p_svh/description/meshes/svh/f13.dae" />
-	</geometry>
-      </collision>
-    </link>
-    <!-- MIDDLE FINGER LINKS -->
-    <link name="${name}_virtual_k">
-      <visual>
-	<origin xyz="0 0 0.01321" />
-	<geometry>
-          <mesh filename="package://schunk_lwa4p_svh/description/meshes/svh/f20.dae" />
-	</geometry>
-      </visual>
-      <collision>
-	<origin xyz="0 0 0.01321" />
-	<geometry>
-          <mesh filename="package://schunk_lwa4p_svh/description/meshes/svh/f20.dae" />
-	</geometry>
-      </collision>
-    </link>
-    <link name="${name}_k">
-      <visual>
-	<geometry>
-          <mesh filename="package://schunk_lwa4p_svh/description/meshes/svh/f21.dae" />
-	</geometry>
-      </visual>
-      <collision>
-	<geometry>
-          <mesh filename="package://schunk_lwa4p_svh/description/meshes/svh/f21.dae" />
-	</geometry>
-      </collision>
-    </link>
-    <link name="${name}_o">
-      <visual>
-	<geometry>
-          <mesh filename="package://schunk_lwa4p_svh/description/meshes/svh/f22.dae" />
-	</geometry>
-      </visual>
-      <collision>
-	<geometry>
-          <mesh filename="package://schunk_lwa4p_svh/description/meshes/svh/f22.dae" />
-	</geometry>
-      </collision>
-    </link>
-    <link name="${name}_s">
-      <visual>
-	<geometry>
-          <mesh filename="package://schunk_lwa4p_svh/description/meshes/svh/f23.dae" />
-	</geometry>
-      </visual>
-      <collision>
-	<geometry>
-          <mesh filename="package://schunk_lwa4p_svh/description/meshes/svh/f23.dae" />
-	</geometry>
-      </collision>
-    </link>
-    <!-- RING FINGER LINKS -->
-    <link name="${name}_virtual_j">
-      <visual>
-	<origin xyz="0 0 -0.01321" />
-	<geometry>
-          <mesh filename="package://schunk_lwa4p_svh/description/meshes/svh/f30.dae" />
-	</geometry>
-      </visual>
-      <collision>
-	<origin xyz="0 0 -0.01321" />
-	<geometry>
-          <mesh filename="package://schunk_lwa4p_svh/description/meshes/svh/f30.dae" />
-	</geometry>
-      </collision>
-    </link>
-    <link name="${name}_j">
-      <visual>
-	<geometry>
-          <mesh filename="package://schunk_lwa4p_svh/description/meshes/svh/f31.dae" />
-	</geometry>
-      </visual>
-      <collision>
-	<geometry>
-          <mesh filename="package://schunk_lwa4p_svh/description/meshes/svh/f31.dae" />
-	</geometry>
-      </collision>
-    </link>
-    <link name="${name}_n">
-      <visual>
-	<geometry>
-          <mesh filename="package://schunk_lwa4p_svh/description/meshes/svh/f32.dae" />
-	</geometry>
-      </visual>
-      <collision>
-	<geometry>
-          <mesh filename="package://schunk_lwa4p_svh/description/meshes/svh/f32.dae" />
-	</geometry>
-      </collision>
-    </link>
-    <link name="${name}_r">
-      <visual>
-	<geometry>
-          <mesh filename="package://schunk_lwa4p_svh/description/meshes/svh/f33.dae" />
-	</geometry>
-      </visual>
-      <collision>
-	<geometry>
-          <mesh filename="package://schunk_lwa4p_svh/description/meshes/svh/f33.dae" />
-	</geometry>
-      </collision>
-    </link>
-    <!-- LITTLE FINGER LINKS -->
-    <link name="${name}_virtual_i">
-      <visual>
-	<origin xyz="0 0 -0.01321" />
-	<geometry>
-          <mesh filename="package://schunk_lwa4p_svh/description/meshes/svh/f40.dae" />
-	</geometry>
-      </visual>
-      <collision>
-	<origin xyz="0 0 -0.01321" />
-	<geometry>
-          <mesh filename="package://schunk_lwa4p_svh/description/meshes/svh/f40.dae" />
-	</geometry>
-      </collision>
-    </link>
-    <link name="${name}_i">
-      <visual>
-	<geometry>
-          <mesh filename="package://schunk_lwa4p_svh/description/meshes/svh/f41.dae" />
-	</geometry>
-      </visual>
-      <collision>
-	<geometry>
-          <mesh filename="package://schunk_lwa4p_svh/description/meshes/svh/f41.dae" />
-	</geometry>
-      </collision>
-    </link>
-    <link name="${name}_m">
-      <visual>
-	<geometry>
-          <mesh filename="package://schunk_lwa4p_svh/description/meshes/svh/f42.dae" />
-	</geometry>
-      </visual>
-      <collision>
-	<geometry>
-          <mesh filename="package://schunk_lwa4p_svh/description/meshes/svh/f42.dae" />
-	</geometry>
-      </collision>
-    </link>
-    <link name="${name}_q">
-      <visual>
-	<geometry>
-          <mesh filename="package://schunk_lwa4p_svh/description/meshes/svh/f43.dae" />
-	</geometry>
-      </visual>
-      <collision>
-	<geometry>
-          <mesh filename="package://schunk_lwa4p_svh/description/meshes/svh/f43.dae" />
-	</geometry>
-      </collision>
-    </link>
-    <joint name="${name}_Thumb_Flexion" type="revolute">
-      <parent link="${name}_virtual_a" />
-      <child link="${name}_a" />
-      <limit effort="1000.0" lower="0.0" upper="0.9704" velocity="1" />
-      <origin xyz="0 0 0" rpy="0 0 ${side*(-0.9704)}" />
-      <axis xyz="0 0 ${side*(1)}" />
-    </joint>
-    <joint name="${name}_Thumb_Helper" type="fixed">
-      <parent link="${name}_z" />
-      <child link="${name}_virtual_a" />
-      <origin xyz="0 0 0.04596" rpy="0 -1.5707 3.1416" />
-    </joint>
-    <!-- BASE_LINE JOINTS -->
-    <joint name="${name}_Thumb_Opposition" type="revolute">
-      <parent link="${name}_e1" />
-      <child link="${name}_z" />
-      <limit effort="1000.0" lower="0.0" upper="0.9879" velocity="1" />
-      <origin xyz="${side*(-0.01690)} 0.02626 0" rpy="0 0.2618 1.571" />
-      <axis xyz="0 0 ${side*(-1)}" />
-    </joint>
-    <!-- JOINT NOT FOR BASE_LINE. BUT WRITTEN DOWN HERE FOR BETTER UX -->
-    <joint name="${name}_f1" type="fixed">
-      <parent link="${name}_e1" />
-      <child link="${name}_d" />
-      <origin xyz="0 0 0" rpy="0 0 0" />
-    </joint>
-    <joint name="${name}_f2" type="fixed">
-      <parent link="${name}_d" />
-      <child link="${name}_h" />
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