Commit message: Added odom to base_link for ekf_localization_node. Ridgeback scanner is running and /front/scan topic does publish data.

File: simulation/grasping_sim/urdf/urdf/ridgeback/ridgeback.urdf.xacro (robot description, xacro)
@@ -100,9 +100,9 @@
       <limit effort="0" velocity="0" />
     </xacro:rocker>
-    <link name="${name}_base_link"></link>
+    <link name="base_link"></link>
     <joint name="base_link_joint" type="fixed">
       <!--<origin xyz="0 0 0" rpy="0 0 0" />-->
       <xacro:insert_block name="origin" />
-      <parent link="${name}_base_link"/>
+      <parent link="base_link"/>
       <child link="chassis_link" />
     </joint>
@@ -262,5 +262,5 @@
     <link name="mid_mount" />
     <joint name="mid_mount_joint" type="fixed" >
-      <parent link="${name}_base_link" />
+      <parent link="base_link" />
       <child link="mid_mount" />
       <origin xyz="0 0 ${deck_height}" rpy="0 0 0"/>
