Commit message: Readme edit

File: simulation/grasping_sim/urdf/robot.urdf.xacro (robot description, xacro)
@@ -80,5 +80,5 @@
       <origin xyz="0 0 0" rpy="0 0 0"/>
       <geometry>
-        <mesh filename="package://zed_wrapper/urdf/models/ZED.stl" />
+        <mesh filename="package://grasping_sim/urdf/urdf/zed/models/ZED.stl" />
       </geometry>
       <material name="light_grey">

Commit message: Generated URDF now contains transmissions for hand joints, links still not showing in gazebo

File: simulation/grasping_sim/urdf/robot.urdf.xacro (robot description, xacro)
@@ -1,4 +1,4 @@
 <?xml version="1.0"?>
-<robot xmlns:xacro="http://www.ros.org/wiki/xacro"
+<robot xmlns:xacro="http://ros.org/wiki/xacro"
        name="lwa4p" >
   <!-- common stuff -->

File: simulation/grasping_sim/urdf/urdf/common.xacro (robot description, xacro)
@@ -1,4 +1,4 @@
 <?xml version="1.0"?>
-<robot xmlns:xacro="http://www.ros.org/wiki/xacro">
+<robot xmlns:xacro="http://ros.org/wiki/xacro">
   <xacro:property name="M_PI" value="3.1415926535897931" />
   <!-- see https://secure.wikimedia.org/wikipedia/en/wiki/List_of_moment_of_inertia_tensors -->

File: simulation/grasping_sim/urdf/urdf/gazebo.urdf.xacro (robot description, xacro)
@@ -1,4 +1,4 @@
 <?xml version="1.0"?>
-<robot xmlns:xacro="http://www.ros.org/wiki/xacro">
+<robot xmlns:xacro="http://ros.org/wiki/xacro">
   <gazebo>
     <plugin name="ros_control" filename="libgazebo_ros_control.so">

File: simulation/grasping_sim/urdf/urdf/lwa4p/lwa4p.gazebo.xacro (robot description, xacro)
@@ -1,4 +1,4 @@
 <?xml version="1.0"?>
-<robot xmlns:xacro="http://www.ros.org/wiki/xacro">
+<robot xmlns:xacro="http://ros.org/wiki/xacro">
   <xacro:macro name="schunk_lwa4p_gazebo" params="name">
     <gazebo reference="${name}_0_link">

File: simulation/grasping_sim/urdf/urdf/lwa4p/lwa4p.transmission.xacro (robot description, xacro)
@@ -1,4 +1,4 @@
 <?xml version="1.0"?>
-<robot xmlns:xacro="http://www.ros.org/wiki/xacro">
+<robot xmlns:xacro="http://ros.org/wiki/xacro">
   <xacro:include filename="$(find grasping_sim)/urdf/urdf/common.xacro" />
   <xacro:macro name="schunk_lwa4p_transmission" params="name">

File: simulation/grasping_sim/urdf/urdf/lwa4p/lwa4p.urdf.xacro (robot description, xacro)
@@ -1,4 +1,4 @@
 <?xml version="1.0"?>
-<robot xmlns:xacro="http://www.ros.org/wiki/xacro">
+<robot xmlns:xacro="http://ros.org/wiki/xacro">
   <xacro:property name="safety_offset" value="0.02"/>
   <xacro:include filename="$(find grasping_sim)/urdf/urdf/common.xacro"/>

File: simulation/grasping_sim/urdf/urdf/svh/svh.transmission.xacro (robot description, xacro)
@@ -1,4 +1,4 @@
 <?xml version="1.0"?>
-<robot xmlns:xacro="http://www.ros.org/wiki/xacro">
+<robot xmlns:xacro="http://ros.org/wiki/xacro">
     <xacro:macro name="svh_transmission" params="name">
         <transmission name="${name}_Finger_Spread_trans">
@@ -57,4 +57,48 @@
             </actuator>
         </transmission>
+        <transmission name="${name}_Index_Finger_Proximal_trans">
+            <type>transmission_interface/SimpleTransmission</type>
+            <joint name="${name}_Index_Finger_Proximal">
+                <hardwareInterface>PositionJointInterface</hardwareInterface>
+                <hardwareInterface>VelocityJointInterface</hardwareInterface>
+                <hardwareInterface>EffortJointInterface</hardwareInterface>
+            </joint>
+            <actuator name="${name}_Index_Finger_Proximal_motor">
+                <mechanicalReduction>1</mechanicalReduction>
+            </actuator>
+        </transmission>
+        <transmission name="${name}_Index_Finger_Distal_trans">
+            <type>transmission_interface/SimpleTransmission</type>
+            <joint name="${name}_Index_Finger_Distal">
+                <hardwareInterface>PositionJointInterface</hardwareInterface>
+                <hardwareInterface>VelocityJointInterface</hardwareInterface>
+                <hardwareInterface>EffortJointInterface</hardwareInterface>
+            </joint>
+            <actuator name="${name}_Index_Finger_Distal_motor">
+                <mechanicalReduction>1</mechanicalReduction>
+            </actuator>
+        </transmission>
+        <transmission name="${name}_Thumb_Flexion_trans">
+            <type>transmission_interface/SimpleTransmission</type>
+            <joint name="${name}_Thumb_Flexion">
+                <hardwareInterface>PositionJointInterface</hardwareInterface>
+                <hardwareInterface>VelocityJointInterface</hardwareInterface>
+                <hardwareInterface>EffortJointInterface</hardwareInterface>
+            </joint>
+            <actuator name="${name}_Thumb_Flexion_motor">
+                <mechanicalReduction>1</mechanicalReduction>
+            </actuator>
+        </transmission>
+        <transmission name="${name}_Thumb_Opposition_trans">
+            <type>transmission_interface/SimpleTransmission</type>
+            <joint name="${name}_Thumb_Opposition">
+                <hardwareInterface>PositionJointInterface</hardwareInterface>
+                <hardwareInterface>VelocityJointInterface</hardwareInterface>
+                <hardwareInterface>EffortJointInterface</hardwareInterface>
+            </joint>
+            <actuator name="${name}_Thumb_Opposition_motor">
+                <mechanicalReduction>1</mechanicalReduction>
+            </actuator>
+        </transmission>
     </xacro:macro>
 </robot>

File: simulation/grasping_sim/urdf/urdf/svh/svh.urdf.xacro (robot description, xacro)
@@ -1,4 +1,4 @@
 <?xml version="1.0"?>
-<robot xmlns:xacro="http://www.ros.org/wiki/xacro">
+<robot xmlns:xacro="http://ros.org/wiki/xacro">
     <xacro:property name="cyl_radius" value="0.001"/>
     <xacro:include filename="$(find grasping_sim)/urdf/urdf/common.xacro"/>
@@ -28,28 +28,28 @@
         </link>
         <link name="${name}_d">
-            <!-- <visual> -->
-            <!-- 	<geometry> -->
-            <!-- 	  <cylinder length="0.110" radius="${cyl_radius}" /> -->
-            <!-- 	</geometry> -->
-            <!-- 	<material name="${name}_green" /> -->
-            <!-- </visual> -->
+             <visual>
+             	<geometry>
+             	  <cylinder length="0.110" radius="${cyl_radius}" />
+             	</geometry>
+             	<material name="${name}_green" />
+             </visual>
         </link>
         <link name="${name}_h">
-            <!-- <visual> -->
-            <!-- 	<origin rpy="0 1.571 0" xyz="${side*(-0.0125)} 0 0.0825" /> -->
-            <!-- 	<geometry> -->
-            <!-- 	  <cylinder length="0.025" radius="${cyl_radius}" /> -->
-            <!-- 	</geometry> -->
-            <!-- 	<material name="${name}_green" /> -->
-            <!-- </visual> -->
+             <visual>
+             	<origin rpy="0 1.571 0" xyz="${side*(-0.0125)} 0 0.0825" />
+             	<geometry>
+             	  <cylinder length="0.025" radius="${cyl_radius}" />
+             	</geometry>
+             	<material name="${name}_green" />
+             </visual>
         </link>
         <link name="${name}_d2">
-            <!-- <visual> -->
-            <!-- 	<origin rpy="0 0 0" xyz="${side*(-0.025)} 0 0.09625" /> -->
-            <!-- 	<geometry> -->
-            <!-- 	  <cylinder length="0.0275" radius="${cyl_radius}" /> -->
-            <!-- 	</geometry> -->
-            <!-- 	<material name="${name}_green" /> -->
-            <!-- </visual> -->
+             <visual>
+             	<origin rpy="0 0 0" xyz="${side*(-0.025)} 0 0.09625" />
+             	<geometry>
+             	  <cylinder length="0.0275" radius="${cyl_radius}" />
+             	</geometry>
+             	<material name="${name}_green" />
+             </visual>
         </link>
         <!-- LENGTH NOT FOUND IN DATASHEET! GUESSED!!! -->
@@ -85,11 +85,11 @@
         <!-- LENGTH NOT FOUND IN DATASHEET! GUESSED!!! -->
         <link name="${name}_e3">
-            <!-- <visual> -->
-            <!-- 	<origin rpy="0 0 0" xyz="${side*(0.0175)} 0 0.015" /> -->
-            <!-- 	<geometry> -->
-            <!-- 	  <cylinder length="0.03" radius="${cyl_radius}" /> -->
-            <!-- 	</geometry> -->
-            <!-- 	<material name="green" /> -->
-            <!-- </visual> -->
+             <visual>
+             	<origin rpy="0 0 0" xyz="${side*(0.0175)} 0 0.015" />
+             	<geometry>
+             	  <cylinder length="0.03" radius="${cyl_radius}" />
+             	</geometry>
+             	<material name="green" />
+             </visual>
         </link>
         <link name="${name}_e">
@@ -97,21 +97,21 @@
         <!-- LENGTH NOT FOUND IN DATASHEET! GUESSED, BUT POSITION CALCULATED: E4 = D-G-F!!! -->
         <link name="${name}_e4">
-            <!-- <visual> -->
-            <!-- 	<origin rpy="0 0 0" xyz="${side*(0.02825)} 0 0.043" /> -->
-            <!-- 	<geometry> -->
-            <!-- 	  <cylinder length="0.026" radius="${cyl_radius}" /> -->
-            <!-- 	</geometry> -->
-            <!-- 	<material name="green" /> -->
-            <!-- </visual> -->
+             <visual>
+             	<origin rpy="0 0 0" xyz="${side*(0.02825)} 0 0.043" />
+             	<geometry>
+             	  <cylinder length="0.026" radius="${cyl_radius}" />
+             	</geometry>
+             	<material name="green" />
+             </visual>
         </link>
         <!-- LENGTH NOT FOUND IN DATASHEET! GUESSED, BUT POSITION CALCULATED: E5 = D-G!!! -->
         <link name="${name}_e5">
-            <!-- <visual> -->
-            <!-- 	<origin rpy="0 0 0" xyz="${side*(0.00675)} 0 0.04775" /> -->
-            <!-- 	<geometry> -->
-            <!-- 	  <cylinder length="0.0355" radius="${cyl_radius}" /> -->
-            <!-- 	</geometry> -->
-            <!-- 	<material name="green" /> -->
-            <!-- </visual> -->
+             <visual>
+             	<origin rpy="0 0 0" xyz="${side*(0.00675)} 0 0.04775" />
+             	<geometry>
+             	  <cylinder length="0.0355" radius="${cyl_radius}" />
+             	</geometry>
+             	<material name="green" />
+             </visual>
         </link>
         <!-- THUMB LINKS -->
@@ -164,5 +164,5 @@
                     <mesh scale="1 ${side*(1)} ${side*(1)}"
                           filename="package://schunk_lwa4p_svh/description/meshes/svh/d13.dae"/>
-                </geometry>
+            (    </geometry>
             </visual>
             <collision>
@@ -587,5 +587,104 @@
         </joint>
         <!-- extensions -->
-    <xacro:svh_transmission name="${name}" />
+    <!--xacro:svh_transmission name="${name}" /-->
+        <transmission name="${name}_Finger_Spread_trans">
+            <type>transmission_interface/SimpleTransmission</type>
+            <joint name="${name}_Finger_Spread">
+                <hardwareInterface>PositionJointInterface</hardwareInterface>
+                <hardwareInterface>VelocityJointInterface</hardwareInterface>
+                <hardwareInterface>EffortJointInterface</hardwareInterface>
+            </joint>
+            <actuator name="${name}_Finger_Spread_motor">
+                <mechanicalReduction>1</mechanicalReduction>
+            </actuator>
+        </transmission>
+        <transmission name="${name}_Pinky_trans">
+            <type>transmission_interface/SimpleTransmission</type>
+            <joint name="${name}_Pinky">
+                <hardwareInterface>PositionJointInterface</hardwareInterface>
+                <hardwareInterface>VelocityJointInterface</hardwareInterface>
+                <hardwareInterface>EffortJointInterface</hardwareInterface>
+            </joint>
+            <actuator name="${name}_Pinky_motor">
+                <mechanicalReduction>1</mechanicalReduction>
+            </actuator>
+        </transmission>
+        <transmission name="${name}_Ring_Finger_trans">
+            <type>transmission_interface/SimpleTransmission</type>
+            <joint name="${name}_Ring_Finger">
+                <hardwareInterface>PositionJointInterface</hardwareInterface>
+                <hardwareInterface>VelocityJointInterface</hardwareInterface>
+                <hardwareInterface>EffortJointInterface</hardwareInterface>
+            </joint>
+            <actuator name="${name}_Ring_Finger_motor">
+                <mechanicalReduction>1</mechanicalReduction>
+            </actuator>
+        </transmission>
+        <transmission name="${name}_Middle_Finger_Proximal_trans">
+            <type>transmission_interface/SimpleTransmission</type>
+            <joint name="${name}_Middle_Finger_Proximal">
+                <hardwareInterface>PositionJointInterface</hardwareInterface>
+                <hardwareInterface>VelocityJointInterface</hardwareInterface>
+                <hardwareInterface>EffortJointInterface</hardwareInterface>
+            </joint>
+            <actuator name="${name}_Middle_Finger_Proximal_motor">
+                <mechanicalReduction>1</mechanicalReduction>
+            </actuator>
+        </transmission>
+        <transmission name="${name}_Middle_Finger_Distal_trans">
+            <type>transmission_interface/SimpleTransmission</type>
+            <joint name="${name}_Middle_Finger_Distal">
+                <hardwareInterface>PositionJointInterface</hardwareInterface>
+                <hardwareInterface>VelocityJointInterface</hardwareInterface>
+                <hardwareInterface>EffortJointInterface</hardwareInterface>
+            </joint>
+            <actuator name="${name}_Middle_Finger_Distal_motor">
+                <mechanicalReduction>1</mechanicalReduction>
+            </actuator>
+        </transmission>
+        <transmission name="${name}_Index_Finger_Proximal_trans">
+            <type>transmission_interface/SimpleTransmission</type>
+            <joint name="${name}_Index_Finger_Proximal">
+                <hardwareInterface>PositionJointInterface</hardwareInterface>
+                <hardwareInterface>VelocityJointInterface</hardwareInterface>
+                <hardwareInterface>EffortJointInterface</hardwareInterface>
+            </joint>
+            <actuator name="${name}_Index_Finger_Proximal_motor">
+                <mechanicalReduction>1</mechanicalReduction>
+            </actuator>
+        </transmission>
+        <transmission name="${name}_Index_Finger_Distal_trans">
+            <type>transmission_interface/SimpleTransmission</type>
+            <joint name="${name}_Index_Finger_Distal">
+                <hardwareInterface>PositionJointInterface</hardwareInterface>
+                <hardwareInterface>VelocityJointInterface</hardwareInterface>
+                <hardwareInterface>EffortJointInterface</hardwareInterface>
+            </joint>
+            <actuator name="${name}_Index_Finger_Distal_motor">
+                <mechanicalReduction>1</mechanicalReduction>
+            </actuator>
+        </transmission>
+        <transmission name="${name}_Thumb_Flexion_trans">
+            <type>transmission_interface/SimpleTransmission</type>
+            <joint name="${name}_Thumb_Flexion">
+                <hardwareInterface>PositionJointInterface</hardwareInterface>
+                <hardwareInterface>VelocityJointInterface</hardwareInterface>
+                <hardwareInterface>EffortJointInterface</hardwareInterface>
+            </joint>
+            <actuator name="${name}_Thumb_Flexion_motor">
+                <mechanicalReduction>1</mechanicalReduction>
+            </actuator>
+        </transmission>
+        <transmission name="${name}_Thumb_Opposition_trans">
+            <type>transmission_interface/SimpleTransmission</type>
+            <joint name="${name}_Thumb_Opposition">
+                <hardwareInterface>PositionJointInterface</hardwareInterface>
+                <hardwareInterface>VelocityJointInterface</hardwareInterface>
+                <hardwareInterface>EffortJointInterface</hardwareInterface>
+            </joint>
+            <actuator name="${name}_Thumb_Opposition_motor">
+                <mechanicalReduction>1</mechanicalReduction>
+            </actuator>
+        </transmission>
     <!-- ros_control plugin -->
     <gazebo>

File: simulation/luh_youbot_description/urdf/sensors/asus_xtion_camera.urdf.xacro (robot description, xacro)
@@ -1,4 +1,4 @@
 <?xml version="1.0"?>
-<robot xmlns:xacro="http://www.ros.org/wiki/xacro">
+<robot xmlns:xacro="http://ros.org/wiki/xacro">
   <xacro:include filename="$(find luh_youbot_description)/urdf/sensors/asus_xtion_camera.gazebo.xacro" />
   <xacro:property name="eye_x_offset" value="0.03" />

Commit message: pushing old updates

File: simulation/grasping_sim/urdf/robot.urdf.xacro (robot description, xacro)
@@ -9,4 +9,6 @@
   <!-- schunk svh -->
   <xacro:include filename="$(find grasping_sim)/urdf/urdf/svh/svh.urdf.xacro" />
+  <!-- schunk sdh -->
+  <xacro:include filename="$(find grasping_sim)/urdf/urdf/sdh/sdh.urdf.xacro" />
   <!-- zed camera -->
 <!--  <xacro:include filename="$(find zed_wrapper)/urdf/zed.urdf"/>-->
@@ -55,7 +57,10 @@
   </xacro:schunk_lwa4p>
   <!-- hand -->
-  <xacro:svh parent="arm_6_link" name="left_hand" side="-1">
-    <origin xyz="0 0 .1"  rpy= "0 0 0" />
-  </xacro:svh>
+<!--  <xacro:svh parent="arm_6_link" name="left_hand" side="-1">-->
+<!--    <origin xyz="0 0 .1"  rpy= "0 0 0" />-->
+<!--  </xacro:svh>-->
+  <xacro:schunk_sdh name="left_hand" parent="arm_6_link">
+    <origin xyz="0 0 0.08"  rpy= "0 0 0"/>
+  </xacro:schunk_sdh>
   <joint name="base_joint" type="fixed">
     <parent link="world"/>

File: simulation/grasping_sim/urdf/urdf/lwa4p/lwa4p.urdf.xacro (robot description, xacro)
@@ -244,7 +244,12 @@
       <plugin name="ros_control" filename="libhwi_switch_gazebo_ros_control.so">
         <robotNamespace>${name}</robotNamespace>
-        <filterJointsParam>joint_names</filterJointsParam>
       </plugin>
     </gazebo>
+<!---->
+<!--    <gazebo>-->
+<!--      <plugin name="gazebo_ros_control" filename="libgazebo_ros_control.so">-->
+<!--        <robotNamespace>${name}</robotNamespace>-->
+<!--      </plugin>-->
+<!--    </gazebo>-->
   </xacro:macro>
 </robot>

File: simulation/grasping_sim/urdf/urdf/sdh/sdh.urdf.xacro (robot description, xacro)
@@ -342,7 +342,12 @@
       <plugin name="ros_control" filename="libhwi_switch_gazebo_ros_control.so">
         <robotNamespace>${name}</robotNamespace>
-        <filterJointsParam>joint_names</filterJointsParam>
       </plugin>
     </gazebo>
+<!---->
+<!--    <gazebo>-->
+<!--      <plugin name="gazebo_ros_control" filename="libgazebo_ros_control.so">-->
+<!--        <robotNamespace>${name}</robotNamespace>-->
+<!--      </plugin>-->
+<!--    </gazebo>-->
   </xacro:macro>
 </robot>

Commit message: Inital commit of branch for two arms with sdh hands.

File: simulation/grasping_sim/urdf/robot.urdf.xacro (robot description, xacro)
@@ -8,5 +8,9 @@
   <xacro:include filename="$(find grasping_sim)/urdf/urdf/lwa4p/lwa4p.urdf.xacro" />
   <!-- schunk svh -->
+  <!--
   <xacro:include filename="$(find grasping_sim)/urdf/urdf/svh/svh.urdf.xacro" />
+  -->
+  <!-- schunk sdh -->
+  <xacro:include filename="$(find grasping_sim)/urdf/urdf/sdh/sdh.urdf.xacro" />
   <!-- zed camera -->
 <!--  <xacro:include filename="$(find zed_wrapper)/urdf/zed.urdf"/>-->
@@ -50,12 +54,26 @@
     <origin xyz=".27 .11 -.67" rpy="0.4887 0 -1.5707"/>
   </joint>
-  <!-- arm -->
-  <xacro:schunk_lwa4p name="arm" parent="body" has_podest="true">
+  <!-- left arm -->
+  <xacro:schunk_lwa4p name="left_arm" parent="body" has_podest="true">
     <origin xyz="0 -0.27 0.08" rpy="1.5707 0 0" /> <!--slightly above gazebo plane-->
   </xacro:schunk_lwa4p>
   <!-- hand -->
+  <!--
   <xacro:svh parent="arm_6_link" name="left_hand" side="-1">
     <origin xyz="0 0 .1"  rpy= "0 0 0" />
   </xacro:svh>
+  -->
+  <!-- left sdh gripper -->
+  <xacro:schunk_sdh name="left_hand" parent="left_arm_6_link">
+    <origin xyz="0 0 0.08"  rpy= "0 0 0"/>
+  </xacro:schunk_sdh>
+   <!-- right arm -->
+   <xacro:schunk_lwa4p name="right_arm" parent="body" has_podest="true">
+     <origin xyz="0 0.18 0.08" rpy="1.5707 0 3.1415" />
+   </xacro:schunk_lwa4p>
+   <!-- right sdh gripper -->
+   <xacro:schunk_sdh name="right_hand" parent="right_arm_6_link">
+    <origin xyz="0 0 0.08"  rpy= "0 0 3.1415"/>
+   </xacro:schunk_sdh>
   <joint name="base_joint" type="fixed">
     <parent link="world"/>

Commit message: Added the sdh hand to the arms.

File: simulation/grasping_sim/urdf/robot.urdf.xacro (robot description, xacro)
@@ -7,8 +7,4 @@
   <!-- schunk lwa4p -->
   <xacro:include filename="$(find grasping_sim)/urdf/urdf/lwa4p/lwa4p.urdf.xacro" />
-  <!-- schunk svh -->
-  <!--
-  <xacro:include filename="$(find grasping_sim)/urdf/urdf/svh/svh.urdf.xacro" />
-  -->
   <!-- schunk sdh -->
   <xacro:include filename="$(find grasping_sim)/urdf/urdf/sdh/sdh.urdf.xacro" />
@@ -55,15 +51,9 @@
   </joint>
   <!-- left arm -->
-  <xacro:schunk_lwa4p name="left_arm" parent="body" has_podest="true">
+  <xacro:schunk_lwa4p name="arm" parent="body" has_podest="true">
     <origin xyz="0 -0.27 0.08" rpy="1.5707 0 0" /> <!--slightly above gazebo plane-->
   </xacro:schunk_lwa4p>
-  <!-- hand -->
-  <!--
-  <xacro:svh parent="arm_6_link" name="left_hand" side="-1">
-    <origin xyz="0 0 .1"  rpy= "0 0 0" />
-  </xacro:svh>
-  -->
-  <!-- left sdh gripper -->
-  <xacro:schunk_sdh name="left_hand" parent="left_arm_6_link">
+  <!-- left sdh hand -->
+  <xacro:schunk_sdh name="left_hand" parent="arm_6_link">
     <origin xyz="0 0 0.08"  rpy= "0 0 0"/>
   </xacro:schunk_sdh>
@@ -179,3 +169,8 @@
     <origin xyz="0.08 -0.04 -0.05" rpy="0 -1.5707 0" />
   </xacro:asus_xtion_camera>
+  <!-- ros_control plugin -->
+  <gazebo>
+    <plugin name="ros_control" filename="libhwi_switch_gazebo_ros_control.so">
+    </plugin>
+  </gazebo>
 </robot>

File: simulation/grasping_sim/urdf/urdf/lwa4p/lwa4p.urdf.xacro (robot description, xacro)
@@ -241,4 +241,5 @@
     <xacro:schunk_lwa4p_transmission name="${name}" />
     <!-- ros_control plugin -->
+    <!--
     <gazebo>
       <plugin name="ros_control" filename="libhwi_switch_gazebo_ros_control.so">
@@ -247,4 +248,5 @@
       </plugin>
     </gazebo>
+    -->
   </xacro:macro>
 </robot>

File: simulation/grasping_sim/urdf/urdf/sdh/sdh.urdf.xacro (robot description, xacro)
@@ -339,9 +339,11 @@
     <xacro:schunk_sdh_transmission name="${name}" />
     <!-- ros_control plugin -->
-    <gazebo>-->
-      <plugin name="ros_control" filename="libhwi_switch_gazebo_ros_control.so">-->
-        <robotNamespace>${name}</robotNamespace>-->
-      </plugin>-->
-    </gazebo>-->
+    <!--
+    <gazebo>
+      <plugin name="ros_control" filename="libhwi_switch_gazebo_ros_control.so">
+        <robotNamespace>${name}</robotNamespace>
+      </plugin>
+     </gazebo>
+     -->
 <!---->
 <!--    <gazebo>-->
