Commit message: Initial commit of the humanoid on the ridgeback with a box as the backlift. Robot now faces positive x-axis direction. Project depends on the ridegeback_description ROS package.

File: simulation/grasping_sim/urdf/robot.urdf.xacro (robot description, xacro)
@@ -9,10 +9,10 @@
   <!-- schunk sdh -->
   <xacro:include filename="$(find grasping_sim)/urdf/urdf/sdh/sdh.urdf.xacro" />
+  <!-- Clearpath Ridgeback -->
+  <xacro:include filename="$(find grasping_sim)/urdf/urdf/ridgeback/ridgeback.urdf.xacro" />
   <!-- zed camera -->
 <!--  <xacro:include filename="$(find zed_wrapper)/urdf/zed.urdf"/>-->
-  <!-- Used for fixing robot to Gazebo -->
-  <link name="world"/>
   <link name="body">
-    <origin xyz="0 0 0" rpy="0 0 0"/>
+    <!-- <origin xyz="0 0 0" rpy="0 0 0"/> -->
     <collision>
 <!--      <origin xyz=".7 .7 -1.33" rpy="1.5707 0 -1.5707"/>-->
@@ -20,5 +20,6 @@
 <!--        <mesh filename="package://schunk_lwa4p_svh/description/meshes/humanoid/chestconvexhull.stl" scale="0.001 0.001 0.001"/>-->
 <!--      </geometry>-->
-      <origin xyz="-0.03 -.046 -0.038" rpy="0 0 0"/>
+      <!--<origin xyz="-0.03 -.046 -0.038" rpy="0 0 0"/>-->
+      <origin xyz="0 0 0" rpy="0 0 0"/>
       <geometry>
         <box size=".4 .525 .576" />
@@ -26,6 +27,13 @@
     </collision>
     <visual>
-      <origin xyz=".7 .7 -1.33" rpy="1.5707 0 -1.5707"/>
-      <geometry>
+      <!-- Origin for box model of body -->
+      <!--<origin xyz="0 0 0" rpy="0 0 0"/> -->
+      <!-- Origin for mesh model of body -->
+      <!--<origin xyz=".7 .7 -1.33" rpy="1.5707 0 -1.5707"/>-->
+      <origin xyz="-0.49 -0.75 -1.0" rpy="${M_PI/2} 0 ${M_PI/2}"/>
+      <geometry>
+        <!-- Box model of body -->
+        <!--<box size="0.4 0.525 0.576" />-->
+        <!-- Mesh model of body -->
         <mesh filename="package://grasping_sim/urdf/meshes/humanoid/chestlowres.stl" scale="0.001 0.001 0.001" />
       </geometry>
@@ -48,25 +56,62 @@
     <parent link="body"/>
     <child link="head"/>
-    <origin xyz=".27 .11 -.67" rpy="0.4887 0 -1.5707"/>
+    <!--<origin xyz=".27 .11 -.67" rpy="0.4887 0 -1.5707"/>-->
+    <origin xyz="0.45 -0.16 -0.35" rpy="0 0 ${M_PI/2}"/>
   </joint>
   <!-- left arm -->
   <xacro:schunk_lwa4p name="arm" parent="body" has_podest="true">
-    <origin xyz="0 -0.27 0.08" rpy="1.5707 0 0" /> <!--slightly above gazebo plane-->
+    <!--<origin xyz="0 -0.27 0.08" rpy="1.5707 0 0" />--> <!--slightly above gazebo plane-->
+    <origin xyz="0.21 0.23 0.42" rpy="${M_PI/2} 0 ${M_PI}" />
   </xacro:schunk_lwa4p>
   <!-- left sdh hand -->
   <xacro:schunk_sdh name="left_hand" parent="arm_6_link">
+    <origin xyz="0 0 0.08"  rpy= "0 0 ${M_PI}"/>
+  </xacro:schunk_sdh>
+  <!-- right arm -->
+  <xacro:schunk_lwa4p name="right_arm" parent="body" has_podest="true">
+    <!--<origin xyz="0 0.18 0.08" rpy="1.5707 0 3.1415" />-->
+    <origin xyz="0.21 -0.24 0.42" rpy="${M_PI/2} 0 0" />
+  </xacro:schunk_lwa4p>
+  <!-- right sdh hand -->
+  <xacro:schunk_sdh name="right_hand" parent="right_arm_6_link">
     <origin xyz="0 0 0.08"  rpy= "0 0 0"/>
   </xacro:schunk_sdh>
-   <!-- right arm -->
-   <xacro:schunk_lwa4p name="right_arm" parent="body" has_podest="true">
-     <origin xyz="0 0.18 0.08" rpy="1.5707 0 3.1415" />
-   </xacro:schunk_lwa4p>
-   <!-- right sdh gripper -->
-   <xacro:schunk_sdh name="right_hand" parent="right_arm_6_link">
-    <origin xyz="0 0 0.08"  rpy= "0 0 3.1415"/>
-   </xacro:schunk_sdh>
-  <joint name="base_joint" type="fixed">
-    <parent link="world"/>
-    <child link="body"/>
+  <!-- ridgeback -->
+  <xacro:clearpath_ridgeback name="ridgeback">
+    <origin xyz="0 0 0" rpy="0 0 0" />
+  </xacro:clearpath_ridgeback>
+  <!-- backlift -->
+  <link name="backlift">
+    <collision>
+      <geometry>
+        <box size="0.1 0.4 0.6" />
+      </geometry>
+      <origin xyz="0 0 0.3" rpy="0 0 0" />
+    </collision>
+    <visual>
+      <geometry>
+        <box size="0.1 0.4 0.6" />
+        <!-- Liftback mesh available but box with prismatic joint may be more useful -->
+        <!--
+        <mesh filename="package://grasping_sim/urdf/meshes/humanoid/backliftlowres.stl" scale="0.001 0.001 0.001" />
+        -->
+      </geometry>
+        <origin xyz="0 0 0.3" rpy="0 0 0" />
+        <!-- Origin if using liftback mesh -->
+        <!-- <origin xyz="0.3 0.75 -0.3" rpy="${M_PI/2} 0 -${M_PI/2}" /> -->
+    </visual>
+  </link>
+  <joint name="ridgeback_backlift" type="fixed">
+    <parent link="ridgeback_top_link" />
+    <child link="backlift" />
+    <origin xyz="-0.2 0 ${deck_height}" rpy="0 0 0" />
+  </joint>
+  <joint name="backlift_body" type="fixed">
+    <parent link="backlift" />
+    <child link="body" />
+    <!-- Origin for box model of body -->
+    <!--<origin xyz="0.25 0 0.6" rpy="0 0 0" />-->
+    <!-- Origin for mesh model of body -->
+    <origin xyz="0 0 0.5" rpy="0 0 0" />
   </joint>
   <joint name="camera_joint" type="fixed">
@@ -163,5 +208,5 @@
     </sensor>
   </gazebo>
-<!-- depth camera -->
+  <!-- depth camera -->
   <!-- Kamera -->
   <xacro:include filename="$(find luh_youbot_description)/urdf/sensors/asus_xtion_camera.urdf.xacro" />

Commit message: Updated body collision origin.

File: simulation/grasping_sim/urdf/robot.urdf.xacro (robot description, xacro)
@@ -21,5 +21,5 @@
 <!--      </geometry>-->
       <!--<origin xyz="-0.03 -.046 -0.038" rpy="0 0 0"/>-->
-      <origin xyz="0 0 0" rpy="0 0 0"/>
+      <origin xyz="-0.49 -0.75 -1.0" rpy="${M_PI/2} 0 ${M_PI/2}"/>
       <geometry>
         <box size=".4 .525 .576" />
@@ -97,7 +97,7 @@
         -->
       </geometry>
-        <origin xyz="0 0 0.3" rpy="0 0 0" />
-        <!-- Origin if using liftback mesh -->
-        <!-- <origin xyz="0.3 0.75 -0.3" rpy="${M_PI/2} 0 -${M_PI/2}" /> -->
+      <origin xyz="0 0 0.3" rpy="0 0 0" />
+      <!-- Origin if using liftback mesh -->
+      <!-- <origin xyz="0.3 0.75 -0.3" rpy="${M_PI/2} 0 -${M_PI/2}" /> -->
     </visual>
   </link>

Commit message: Updated body collision origin.

File: simulation/grasping_sim/urdf/robot.urdf.xacro (robot description, xacro)
@@ -21,7 +21,7 @@
 <!--      </geometry>-->
       <!--<origin xyz="-0.03 -.046 -0.038" rpy="0 0 0"/>-->
-      <origin xyz="-0.49 -0.75 -1.0" rpy="${M_PI/2} 0 ${M_PI/2}"/>
-      <geometry>
-        <box size=".4 .525 .576" />
+      <origin xyz="0 0 0" rpy="0 0 0"/>
+      <geometry>
+        <box size="0.4 0.525 0.576" />
       </geometry>
     </collision>

Commit message: Added velocity control to the ridgeback to move the humanoid.

File: simulation/grasping_sim/urdf/robot.urdf.xacro (robot description, xacro)
@@ -40,4 +40,7 @@
     </visual>
   </link>
+  <gazebo reference="body">
+    <material>Gazebo/Gold</material>
+  </gazebo>
   <link name="head">
     <origin xyz="0 0 0" rpy="0 0 0"/>
@@ -53,4 +56,7 @@
     </visual>
   </link>
+  <gazebo reference="head">
+    <material>Gazebo/Grey</material>
+  </gazebo>
   <joint name="head_neck" type="fixed">
     <parent link="body"/>
@@ -64,4 +70,19 @@
     <origin xyz="0.21 0.23 0.42" rpy="${M_PI/2} 0 ${M_PI}" />
   </xacro:schunk_lwa4p>
+  <gazebo reference="arm_1_link">
+    <material>Gazebo/Yellow</material>
+  </gazebo>
+  <gazebo reference="arm_2_link">
+    <material>Gazebo/SkyBlue</material>
+  </gazebo>
+  <gazebo reference="arm_3_link">
+    <material>Gazebo/Yellow</material>
+  </gazebo>
+  <gazebo reference="arm_4_link">
+    <material>Gazebo/SkyBlue</material>
+  </gazebo>
+  <gazebo reference="arm_5_link">
+    <material>Gazebo/Yellow</material>
+  </gazebo>
   <!-- left sdh hand -->
   <xacro:schunk_sdh name="left_hand" parent="arm_6_link">
@@ -73,4 +94,19 @@
     <origin xyz="0.21 -0.24 0.42" rpy="${M_PI/2} 0 0" />
   </xacro:schunk_lwa4p>
+  <gazebo reference="right_arm_1_link">
+    <material>Gazebo/Yellow</material>
+  </gazebo>
+  <gazebo reference="right_arm_2_link">
+    <material>Gazebo/SkyBlue</material>
+  </gazebo>
+  <gazebo reference="right_arm_3_link">
+    <material>Gazebo/Yellow</material>
+  </gazebo>
+  <gazebo reference="right_arm_4_link">
+    <material>Gazebo/SkyBlue</material>
+  </gazebo>
+  <gazebo reference="right_arm_5_link">
+    <material>Gazebo/Yellow</material>
+  </gazebo>
   <!-- right sdh hand -->
   <xacro:schunk_sdh name="right_hand" parent="right_arm_6_link">
@@ -92,5 +128,5 @@
       <geometry>
         <box size="0.1 0.4 0.6" />
-        <!-- Liftback mesh available but box with prismatic joint may be more useful -->
+        <!-- Backlift mesh available but box with prismatic joint may be more useful -->
         <!--
         <mesh filename="package://grasping_sim/urdf/meshes/humanoid/backliftlowres.stl" scale="0.001 0.001 0.001" />
@@ -98,8 +134,11 @@
       </geometry>
       <origin xyz="0 0 0.3" rpy="0 0 0" />
-      <!-- Origin if using liftback mesh -->
+      <!-- Origin if using backlift mesh -->
       <!-- <origin xyz="0.3 0.75 -0.3" rpy="${M_PI/2} 0 -${M_PI/2}" /> -->
     </visual>
   </link>
+  <gazebo reference="backlift">
+    <material>Gazebo/DarkGrey</material>
+  </gazebo>
   <joint name="ridgeback_backlift" type="fixed">
     <parent link="ridgeback_top_link" />
@@ -113,4 +152,6 @@
     <!--<origin xyz="0.25 0 0.6" rpy="0 0 0" />-->
     <!-- Origin for mesh model of body -->
+    <axis xyz="0 0 1" />
+    <limit effort="10.0" lower="-0.3" upper="0.1" velocity="0.2" />
     <origin xyz="0 0 0.5" rpy="0 0 0" />
   </joint>

File: simulation/grasping_sim/urdf/urdf/ridgeback/ridgeback.urdf.xacro (robot description, xacro)
@@ -266,4 +266,16 @@
       <origin xyz="0 0 ${deck_height}" rpy="0 0 0"/>
     </joint>
+    <!-- Individual link colouring still needed in Gazebo 2.x -->
+    <gazebo reference="chassis_link"><material>Gazebo/DarkGrey</material></gazebo>
+    <gazebo reference="${name}_top_link"><material>Gazebo/DarkGrey</material></gazebo>
+    <gazebo reference="left_side_cover_link"><material>Gazebo/Yellow</material></gazebo>
+    <gazebo reference="right_side_cover_link"><material>Gazebo/Yellow</material></gazebo>
+    <gazebo reference="front_cover_link"><material>Gazebo/DarkGrey</material></gazebo>
+    <gazebo reference="rear_cover_link"><material>Gazebo/DarkGrey</material></gazebo>
+    <gazebo reference="front_lights_link"><material>Gazebo/WhiteGlow</material></gazebo>
+    <gazebo reference="rear_lights_link"><material>Gazebo/RedGlow</material></gazebo>
+    <gazebo reference="front_rocker_link"><material>Gazebo/DarkGrey</material></gazebo>
+    <gazebo reference="rear_rocker_link"><material>Gazebo/DarkGrey</material></gazebo>
+    <gazebo reference="axle_link"><material>Gazebo/DarkGrey</material></gazebo>
     <!-- Bring in simulation data for Gazebo. -->
     <!--

Commit message: Updated backlift to be a prismatic joint to control the height of the humanoid.

File: simulation/grasping_sim/urdf/robot.urdf.xacro (robot description, xacro)
@@ -121,5 +121,5 @@
     <collision>
       <geometry>
-        <box size="0.1 0.4 0.6" />
+        <box size="0.1 0.4 0.8" />
       </geometry>
       <origin xyz="0 0 0.3" rpy="0 0 0" />
@@ -127,5 +127,5 @@
     <visual>
       <geometry>
-        <box size="0.1 0.4 0.6" />
+        <box size="0.1 0.4 0.8" />
         <!-- Backlift mesh available but box with prismatic joint may be more useful -->
         <!--
@@ -137,4 +137,12 @@
       <!-- <origin xyz="0.3 0.75 -0.3" rpy="${M_PI/2} 0 -${M_PI/2}" /> -->
     </visual>
+    <inertial>
+      <origin xyz="0 0 0" rpy="0 0 0" />
+      <mass value="1" />
+      <inertia
+              ixx="1.0" ixy="0.0" ixz="0.0"
+              iyy="1.0" iyz="0.0"
+              izz="1.0" />
+    </inertial>
   </link>
   <gazebo reference="backlift">
@@ -146,5 +154,5 @@
     <origin xyz="-0.2 0 ${deck_height}" rpy="0 0 0" />
   </joint>
-  <joint name="backlift_body" type="fixed">
+  <joint name="backlift_body" type="prismatic">
     <parent link="backlift" />
     <child link="body" />
@@ -153,7 +161,17 @@
     <!-- Origin for mesh model of body -->
     <axis xyz="0 0 1" />
-    <limit effort="10.0" lower="-0.3" upper="0.1" velocity="0.2" />
+    <limit effort="100.0" lower="-0.4" upper="0.1" velocity="0.1" />
     <origin xyz="0 0 0.5" rpy="0 0 0" />
   </joint>
+  <!-- Backlift and body transmission -->
+  <transmission name="backlift_body_trans">
+    <type>transmission_interface/SimpleTransmission</type>
+    <joint name="backlift_body">
+      <hardwareInterface>hardware_interface/PositionJointInterface</hardwareInterface>
+    </joint>
+    <actuator name="backlift_motor">
+      <mechanicalReduction>1</mechanicalReduction>
+    </actuator>
+  </transmission>
   <joint name="camera_joint" type="fixed">
     <parent link="head"/>

Commit message: Made the joint between the body and head to be revolute.

File: simulation/grasping_sim/urdf/robot.urdf.xacro (robot description, xacro)
@@ -54,4 +54,5 @@
         <mesh filename="package://grasping_sim/urdf/meshes/humanoid/headlowres.stl" scale="0.001 0.001 0.001" />
       </geometry>
+      <origin xyz="0.2 -0.16 -1.05" rpy="0 0 ${M_PI/2}"/>
     </visual>
   </link>
@@ -59,10 +60,23 @@
     <material>Gazebo/Grey</material>
   </gazebo>
-  <joint name="head_neck" type="fixed">
+  <joint name="head_neck" type="revolute">
     <parent link="body"/>
     <child link="head"/>
     <!--<origin xyz=".27 .11 -.67" rpy="0.4887 0 -1.5707"/>-->
-    <origin xyz="0.45 -0.16 -0.35" rpy="0 0 ${M_PI/2}"/>
-  </joint>
+    <!--<origin xyz="0.45 -0.16 -0.35" rpy="0 0 ${M_PI/2}"/> -->
+    <origin xyz="0.24 0.0 0.69" rpy="0 0 0"/>
+    <axis xyz="0 1 0" /> <!-- Seems like it should be the y axis not the x axis -->
+    <limit effort="10" velocity="0.25" lower="-0.3" upper="0.4" />
+  </joint>
+  <!-- Transmission for the neck -->
+  <transmission name="head_neck_trans">
+    <type>transmission_interface/SimpleTransmission</type>
+    <actuator name="$head_neck_motor">
+      <mechanicalReduction>1</mechanicalReduction>
+    </actuator>
+    <joint name="head_neck">
+      <hardwareInterface>hardware_interface/PositionJointInterface</hardwareInterface>
+    </joint>
+  </transmission>
   <!-- left arm -->
   <xacro:schunk_lwa4p name="arm" parent="body" has_podest="true">
@@ -190,5 +204,6 @@
   <link name="zed_camera_center">
     <visual>
-      <origin xyz="0 0 0" rpy="0 0 0"/>
+      <!-- <origin xyz="0 0 0" rpy="0 0 0"/> -->
+      <origin xyz="0.034 0.02 -1.05" rpy="0 0 ${M_PI/2}"/> <!-- x increase moves it right -->
       <geometry>
         <mesh filename="package://grasping_sim/urdf/urdf/zed/models/ZED.stl" />
@@ -276,4 +291,5 @@
   <gazebo>
     <plugin name="ros_control" filename="libhwi_switch_gazebo_ros_control.so">
+      <robotNamespace></robotNamespace>
     </plugin>
   </gazebo>

Commit message: Moved backlift to the center of the Ridgeback platform.

File: simulation/grasping_sim/urdf/robot.urdf.xacro (robot description, xacro)
@@ -166,5 +166,5 @@
     <parent link="ridgeback_top_link" />
     <child link="backlift" />
-    <origin xyz="-0.2 0 ${deck_height}" rpy="0 0 0" />
+    <origin xyz="0.0 0 ${deck_height}" rpy="0 0 0" />
   </joint>
   <joint name="backlift_body" type="prismatic">

Commit message: Test simple robot.

File: simulation/grasping_sim/urdf/robot.urdf.xacro (robot description, xacro)
@@ -39,4 +39,9 @@
       </geometry>
     </visual>
+    <inertial>
+        <origin xyz="0 0 0.5" rpy="0 0 0" />
+        <mass value="2" />
+        <inertia ixx="0.05" ixy="0.0" ixz="0.0" iyy="0.05" iyz="0.0" izz="0.05" />
+    </inertial>
   </link>
   <gazebo reference="body">
@@ -56,4 +61,9 @@
       <origin xyz="0.2 -0.16 -1.05" rpy="0 0 ${M_PI/2}"/>
     </visual>
+    <inertial>
+        <origin xyz="0 0 0.05" rpy="0 0 0" />
+        <mass value="0.5" />
+        <inertia ixx="0.01" ixy="0.0" ixz="0.0" iyy="0.01" iyz="0.0" izz="0.01" />
+    </inertial>
   </link>
   <gazebo reference="head">
@@ -81,5 +91,4 @@
   <!-- left arm -->
   <xacro:schunk_lwa4p name="arm" parent="body" has_podest="true">
-    <!--<origin xyz="0 -0.27 0.08" rpy="1.5707 0 0" />--> <!--slightly above gazebo plane-->
     <origin xyz="0.21 0.23 0.42" rpy="${M_PI/2} 0 ${M_PI}" />
   </xacro:schunk_lwa4p>
@@ -105,5 +114,4 @@
   <!-- right arm -->
   <xacro:schunk_lwa4p name="right_arm" parent="body" has_podest="true">
-    <!--<origin xyz="0 0.18 0.08" rpy="1.5707 0 3.1415" />-->
     <origin xyz="0.21 -0.24 0.42" rpy="${M_PI/2} 0 0" />
   </xacro:schunk_lwa4p>
@@ -137,5 +145,5 @@
         <box size="0.1 0.4 0.8" />
       </geometry>
-      <origin xyz="0 0 0.3" rpy="0 0 0" />
+      <origin xyz="0 0 0.4" rpy="0 0 0" />
     </collision>
     <visual>
@@ -147,15 +155,15 @@
         -->
       </geometry>
-      <origin xyz="0 0 0.3" rpy="0 0 0" />
+      <origin xyz="0 0 0.4" rpy="0 0 0" />
       <!-- Origin if using backlift mesh -->
       <!-- <origin xyz="0.3 0.75 -0.3" rpy="${M_PI/2} 0 -${M_PI/2}" /> -->
     </visual>
     <inertial>
-      <origin xyz="0 0 0" rpy="0 0 0" />
+      <origin xyz="0 0 0.2" rpy="0 0 0" />
       <mass value="1" />
       <inertia
-              ixx="1.0" ixy="0.0" ixz="0.0"
-              iyy="1.0" iyz="0.0"
-              izz="1.0" />
+              ixx="0.01" ixy="0.0" ixz="0.0"
+              iyy="0.01" iyz="0.0"
+              izz="0.01" />
     </inertial>
   </link>

File: simulation/grasping_sim/urdf/urdf/ridgeback/ridgeback.urdf.xacro (robot description, xacro)
@@ -282,4 +282,5 @@
     <xacro:include filename="$(find ridgeback_description)/urdf/ridgeback.gazebo" />
     -->
+    <xacro:include filename="$(find grasping_sim)/urdf/ridgeback.gazebo" />
     <!-- Optional standard accessories, including their simulation data. The rendering
          of these into the final description is controlled by optenv variables, which

Commit message: Fixed arms, backlift, and neck controller manager to be one node.

File: simulation/grasping_sim/urdf/robot.urdf.xacro (robot description, xacro)
@@ -39,9 +39,4 @@
       </geometry>
     </visual>
-    <inertial>
-        <origin xyz="0 0 0.5" rpy="0 0 0" />
-        <mass value="2" />
-        <inertia ixx="0.05" ixy="0.0" ixz="0.0" iyy="0.05" iyz="0.0" izz="0.05" />
-    </inertial>
   </link>
   <gazebo reference="body">
@@ -61,9 +56,4 @@
       <origin xyz="0.2 -0.16 -1.05" rpy="0 0 ${M_PI/2}"/>
     </visual>
-    <inertial>
-        <origin xyz="0 0 0.05" rpy="0 0 0" />
-        <mass value="0.5" />
-        <inertia ixx="0.01" ixy="0.0" ixz="0.0" iyy="0.01" iyz="0.0" izz="0.01" />
-    </inertial>
   </link>
   <gazebo reference="head">
@@ -73,8 +63,7 @@
     <parent link="body"/>
     <child link="head"/>
-    <!--<origin xyz=".27 .11 -.67" rpy="0.4887 0 -1.5707"/>-->
     <!--<origin xyz="0.45 -0.16 -0.35" rpy="0 0 ${M_PI/2}"/> -->
     <origin xyz="0.24 0.0 0.69" rpy="0 0 0"/>
-    <axis xyz="0 1 0" /> <!-- Seems like it should be the y axis not the x axis -->
+    <axis xyz="0 1 0" />
     <limit effort="10" velocity="0.25" lower="-0.3" upper="0.4" />
   </joint>
@@ -91,4 +80,5 @@
   <!-- left arm -->
   <xacro:schunk_lwa4p name="arm" parent="body" has_podest="true">
+    <!--<origin xyz="0 -0.27 0.08" rpy="1.5707 0 0" />--> <!--slightly above gazebo plane-->
     <origin xyz="0.21 0.23 0.42" rpy="${M_PI/2} 0 ${M_PI}" />
   </xacro:schunk_lwa4p>
@@ -114,4 +104,5 @@
   <!-- right arm -->
   <xacro:schunk_lwa4p name="right_arm" parent="body" has_podest="true">
+    <!--<origin xyz="0 0.18 0.08" rpy="1.5707 0 3.1415" />-->
     <origin xyz="0.21 -0.24 0.42" rpy="${M_PI/2} 0 0" />
   </xacro:schunk_lwa4p>
@@ -145,5 +136,5 @@
         <box size="0.1 0.4 0.8" />
       </geometry>
-      <origin xyz="0 0 0.4" rpy="0 0 0" />
+      <origin xyz="0 0 0.3" rpy="0 0 0" />
     </collision>
     <visual>
@@ -155,15 +146,15 @@
         -->
       </geometry>
-      <origin xyz="0 0 0.4" rpy="0 0 0" />
+      <origin xyz="0 0 0.3" rpy="0 0 0" />
       <!-- Origin if using backlift mesh -->
       <!-- <origin xyz="0.3 0.75 -0.3" rpy="${M_PI/2} 0 -${M_PI/2}" /> -->
     </visual>
     <inertial>
-      <origin xyz="0 0 0.2" rpy="0 0 0" />
+      <origin xyz="0 0 0" rpy="0 0 0" />
       <mass value="1" />
       <inertia
-              ixx="0.01" ixy="0.0" ixz="0.0"
-              iyy="0.01" iyz="0.0"
-              izz="0.01" />
+              ixx="1.0" ixy="0.0" ixz="0.0"
+              iyy="1.0" iyz="0.0"
+              izz="1.0" />
     </inertial>
   </link>
@@ -174,5 +165,5 @@
     <parent link="ridgeback_top_link" />
     <child link="backlift" />
-    <origin xyz="0.0 0 ${deck_height}" rpy="0 0 0" />
+    <origin xyz="0 0 ${deck_height}" rpy="0 0 0" />
   </joint>
   <joint name="backlift_body" type="prismatic">
@@ -212,5 +203,5 @@
   <link name="zed_camera_center">
     <visual>
-      <!-- <origin xyz="0 0 0" rpy="0 0 0"/> -->
+       <!-- <origin xyz="0 0 0" rpy="0 0 0"/> -->
       <origin xyz="0.034 0.02 -1.05" rpy="0 0 ${M_PI/2}"/> <!-- x increase moves it right -->
       <geometry>
@@ -299,5 +290,5 @@
   <gazebo>
     <plugin name="ros_control" filename="libhwi_switch_gazebo_ros_control.so">
-      <robotNamespace></robotNamespace>
+    <robotNamespace></robotNamespace>
     </plugin>
   </gazebo>

File: simulation/grasping_sim/urdf/urdf/ridgeback/ridgeback.urdf.xacro (robot description, xacro)
@@ -282,5 +282,4 @@
     <xacro:include filename="$(find ridgeback_description)/urdf/ridgeback.gazebo" />
     -->
-    <xacro:include filename="$(find grasping_sim)/urdf/ridgeback.gazebo" />
     <!-- Optional standard accessories, including their simulation data. The rendering
          of these into the final description is controlled by optenv variables, which
