Commit message: Set camera_joint origin to xyz=0 0 0 rpy=0 0 0 so that the position for ZED and Asus Xtion cameras is easier to adjust. Asus xtion camera placed in same position as ZED.

File: simulation/grasping_sim/urdf/robot.urdf.xacro (robot description, xacro)
@@ -190,5 +190,6 @@
     <parent link="head"/>
     <child link="zed_base_link"/>
-    <origin xyz=".155 0.03 1.14" rpy="0 0 -1.5707" />
+    <!-- <origin xyz=".155 0.03 1.14" rpy="0 0 -1.5707" /> -->
+    <origin xyz="0.0 0.0 0.0" rpy="0 0 0" />
   </joint>
   <!-- base_link -->
@@ -203,6 +204,5 @@
   <link name="zed_camera_center">
     <visual>
-       <!-- <origin xyz="0 0 0" rpy="0 0 0"/> -->
-      <origin xyz="0.034 0.02 -1.05" rpy="0 0 ${M_PI/2}"/> <!-- x increase moves it right -->
+      <origin xyz="0.17 -0.005 0.09" rpy="0 0 0"/>
       <geometry>
         <mesh filename="package://grasping_sim/urdf/urdf/zed/models/ZED.stl" />
@@ -217,14 +217,14 @@
     <parent link="zed_camera_center"/>
     <child link="zed_left_camera_frame"/>
-    <origin xyz="0 0.06 0" rpy="0 0 0" />
+    <origin xyz="0 0.0 0" rpy="0 0 0" />
   </joint>
   <link name="zed_left_camera_frame" />
   <joint name="zed_left_camera_depth_joint" type="fixed">
-    <origin xyz="0.05 0.05 0.05" rpy="-1.5707 1.5707 -1.5707"/>
+    <origin xyz="0.0 0.0 0.0" rpy="0 0 0"/>
     <parent link="zed_left_camera_frame"/>
     <child link="zed_depth_frame"/>
   </joint>
   <joint name="zed_left_camera_optical_joint" type="fixed">
-    <origin xyz="0 0 0" rpy="-1.57079632679 0.0 -1.57079632679"/>
+    <origin xyz="0 0 0.0" rpy="0 0.0 0"/>
     <parent link="zed_left_camera_frame"/>
     <child link="zed_left_camera_optical_frame"/>
@@ -249,5 +249,5 @@
       <update_rate>15.0</update_rate>
       <camera name="head">
-        <pose>0.005 0 0 0 0 0</pose>
+        <pose>0.175 0 0.089 0 0 0.0</pose>
         <horizontal_fov>1.3962634</horizontal_fov>
         <image>
@@ -285,5 +285,6 @@
   <xacro:include filename="$(find luh_youbot_description)/urdf/sensors/asus_xtion_camera.urdf.xacro" />
   <xacro:asus_xtion_camera name="camera" parent="zed_depth_frame" tilt="0.0">
-    <origin xyz="0.08 -0.04 -0.05" rpy="0 -1.5707 0" />
+    <!-- <origin xyz="0.08 -0.04 -0.05" rpy="0 -1.5707 0" /> -->
+    <origin xyz="0.16 -0.01 0.053" rpy="0 0 0" /> <!-- Same position as ZED camera -->
   </xacro:asus_xtion_camera>
   <!-- ros_control plugin -->

File: simulation/luh_youbot_description/urdf/sensors/asus_xtion_camera.urdf.xacro (robot description, xacro)
@@ -25,11 +25,11 @@
         <inertia ixx="0.0001" ixy="0" ixz="0" iyy="0.0001" iyz="0" izz="0.0001" />
       </inertial>
-<!--      <visual>-->
-<!--        <origin xyz="0.01 0 0" rpy="${M_PI/2} 0 ${M_PI/2}" />-->
-<!--        <geometry>-->
-<!--           <mesh filename="package://luh_youbot_description/meshes/sensors/asus_xtion_pro_live_base.dae" scale="0.0004 0.0007 0.001"/>-->
-<!--        </geometry>-->
-<!--        <material name="Black" />-->
-<!--      </visual>-->
+     <!-- <visual>
+        <origin xyz="0.01 0 0" rpy="${M_PI/2} 0 ${M_PI/2}" />
+        <geometry>
+           <mesh filename="package://luh_youbot_description/meshes/sensors/asus_xtion_pro_live_base.dae" scale="0.0004 0.0007 0.001"/>
+        </geometry>
+        <material name="Black" />
+      </visual> -->
 <!--      <collision>-->
 <!--        <origin xyz="0.01 0 0" rpy="${M_PI/2} 0 ${M_PI/2}" />-->
@@ -50,11 +50,11 @@
         <inertia ixx="0.0001" ixy="0" ixz="0" iyy="0.0001" iyz="0" izz="0.0001" />
       </inertial>
-<!--      <visual>-->
-<!--        <origin xyz="0 0 0.0075" rpy="0 0 0" />-->
-<!--        <geometry>-->
-<!--          <cylinder length="0.025" radius="0.005" />-->
-<!--        </geometry>-->
-<!--        <material name="Black" />-->
-<!--      </visual>-->
+      <!-- <visual>
+        <origin xyz="0 0 0.0075" rpy="0 0 0" />
+        <geometry>
+         <cylinder length="0.025" radius="0.005" />
+       </geometry>
+       <material name="Black" />
+     </visual> -->
 <!--      <collision>-->
 <!--        <origin xyz="0 0 0.0075" rpy="0 0 0" />-->
@@ -72,4 +72,5 @@
 		<!--<limit effort="100" lower="-0.541052068" upper="0.541052068" velocity="1.0"/>-->
     </joint>
+    <!-- Camera Body-->
     <link name="${name}_camera">
       <inertial>
@@ -78,11 +79,11 @@
         <inertia ixx="0.0001" ixy="0" ixz="0" iyy="0.0001" iyz="0" izz="0.0001" />
       </inertial>
-<!--      <visual>-->
-<!--        <origin xyz="0.02 -0.03 0" rpy="${M_PI/2} 0 ${M_PI/2}" />-->
-<!--        <geometry>-->
-<!--          <mesh filename="package://luh_youbot_description/meshes/sensors/asus_xtion_pro_live_camera.dae" scale="0.001 0.001 0.001"/>-->
-<!--        </geometry>-->
-<!--        <material name="Black" />-->
-<!--      </visual>-->
+      <!-- <visual>
+       <origin xyz="0.02 -0.03 0" rpy="${M_PI/2} 0 ${M_PI/2}" />
+       <geometry>
+         <mesh filename="package://luh_youbot_description/meshes/sensors/asus_xtion_pro_live_camera.dae" scale="0.001 0.001 0.001"/>
+       </geometry>
+       <material name="Black" />
+      </visual> -->
 <!--      <collision>-->
 <!--        <origin xyz="0.02 -0.03 0" rpy="${M_PI/2} 0 ${M_PI/2}" />-->

Commit message: Commented out the visual section of the zed_camera_center to make it invisible.

File: simulation/grasping_sim/urdf/robot.urdf.xacro (robot description, xacro)
@@ -202,5 +202,6 @@
     <origin xyz="0 0 0" rpy="0 0 0" />
   </joint>
-  <link name="zed_camera_center">
+  <link name="zed_camera_center"> <!-- Commented out to allow multiple cameras to see out head visor. -->
+  <!--
     <visual>
       <origin xyz="0.17 -0.005 0.09" rpy="0 0 0"/>
@@ -212,4 +213,5 @@
       </material>
     </visual>
+    -->
   </link>
   <!-- Left Camera -->

File: simulation/grasping_sim/urdf/two_arm_robot.urdf.xacro (robot description, xacro)
@@ -145,5 +145,6 @@
     <origin xyz="0 0 0" rpy="0 0 0" />
   </joint>
-  <link name="zed_camera_center">
+  <link name="zed_camera_center"> <!-- Commented out to allow multiple cameras to see out head visor. -->
+  <!--
     <visual>
       <origin xyz="0.17 -0.005 0.09" rpy="0 0 0"/>
@@ -155,4 +156,5 @@
       </material>
     </visual>
+    -->
   </link>
   <!-- Left Camera -->

Commit message: Moved full formed humanoid to seperate launch and xacro files called full_humanoid_gazebo.launch and full_robot.urdf.xacro.

File: simulation/grasping_sim/urdf/robot.urdf.xacro (robot description, xacro)
@@ -9,10 +9,10 @@
   <!-- schunk sdh -->
   <xacro:include filename="$(find grasping_sim)/urdf/urdf/sdh/sdh.urdf.xacro" />
-  <!-- Clearpath Ridgeback -->
-  <xacro:include filename="$(find grasping_sim)/urdf/urdf/ridgeback/ridgeback.urdf.xacro" />
   <!-- zed camera -->
 <!--  <xacro:include filename="$(find zed_wrapper)/urdf/zed.urdf"/>-->
+  <!-- Used for fixing robot to Gazebo -->
+  <link name="world"/>
   <link name="body">
-    <!-- <origin xyz="0 0 0" rpy="0 0 0"/> -->
+    <origin xyz="0 0 0" rpy="0 0 0"/>
     <collision>
 <!--      <origin xyz=".7 .7 -1.33" rpy="1.5707 0 -1.5707"/>-->
@@ -20,27 +20,16 @@
 <!--        <mesh filename="package://schunk_lwa4p_svh/description/meshes/humanoid/chestconvexhull.stl" scale="0.001 0.001 0.001"/>-->
 <!--      </geometry>-->
-      <!--<origin xyz="-0.03 -.046 -0.038" rpy="0 0 0"/>-->
-      <origin xyz="0 0 0" rpy="0 0 0"/>
+      <origin xyz="-0.03 -.046 -0.038" rpy="0 0 0"/>
       <geometry>
-        <box size="0.4 0.525 0.576" />
+        <box size=".4 .525 .576" />
       </geometry>
     </collision>
     <visual>
-      <!-- Origin for box model of body -->
-      <!--<origin xyz="0 0 0" rpy="0 0 0"/> -->
-      <!-- Origin for mesh model of body -->
-      <!--<origin xyz=".7 .7 -1.33" rpy="1.5707 0 -1.5707"/>-->
-      <origin xyz="-0.49 -0.75 -1.0" rpy="${M_PI/2} 0 ${M_PI/2}"/>
+      <origin xyz=".7 .7 -1.33" rpy="1.5707 0 -1.5707"/>
       <geometry>
-        <!-- Box model of body -->
-        <!--<box size="0.4 0.525 0.576" />-->
-        <!-- Mesh model of body -->
         <mesh filename="package://grasping_sim/urdf/meshes/humanoid/chestlowres.stl" scale="0.001 0.001 0.001" />
       </geometry>
     </visual>
   </link>
-  <gazebo reference="body">
-    <material>Gazebo/Gold</material>
-  </gazebo>
   <link name="head">
     <origin xyz="0 0 0" rpy="0 0 0"/>
@@ -54,142 +43,35 @@
         <mesh filename="package://grasping_sim/urdf/meshes/humanoid/headlowres.stl" scale="0.001 0.001 0.001" />
       </geometry>
-      <origin xyz="0.2 -0.16 -1.05" rpy="0 0 ${M_PI/2}"/>
     </visual>
   </link>
-  <gazebo reference="head">
-    <material>Gazebo/Grey</material>
-  </gazebo>
-  <joint name="head_neck" type="revolute">
+  <joint name="head_neck" type="fixed">
     <parent link="body"/>
     <child link="head"/>
-    <!--<origin xyz="0.45 -0.16 -0.35" rpy="0 0 ${M_PI/2}"/> -->
-    <origin xyz="0.24 0.0 0.69" rpy="0 0 0"/>
-    <axis xyz="0 1 0" />
-    <limit effort="10" velocity="0.25" lower="-0.3" upper="0.4" />
+    <origin xyz=".27 .11 -.67" rpy="0.4887 0 -1.5707"/>
   </joint>
-  <!-- Transmission for the neck -->
-  <transmission name="head_neck_trans">
-    <type>transmission_interface/SimpleTransmission</type>
-    <actuator name="$head_neck_motor">
-      <mechanicalReduction>1</mechanicalReduction>
-    </actuator>
-    <joint name="head_neck">
-      <hardwareInterface>hardware_interface/PositionJointInterface</hardwareInterface>
-    </joint>
-  </transmission>
   <!-- left arm -->
-  <xacro:schunk_lwa4p name="arm" parent="body" has_podest="true">
-    <!--<origin xyz="0 -0.27 0.08" rpy="1.5707 0 0" />--> <!--slightly above gazebo plane-->
-    <origin xyz="0.21 0.23 0.42" rpy="${M_PI/2} 0 ${M_PI}" />
+  <xacro:schunk_lwa4p name="left_arm" parent="body" has_podest="true">
+    <origin xyz="0 -0.27 0.08" rpy="1.5707 0 0" /> <!--slightly above gazebo plane-->
   </xacro:schunk_lwa4p>
-  <gazebo reference="arm_1_link">
-    <material>Gazebo/Yellow</material>
-  </gazebo>
-  <gazebo reference="arm_2_link">
-    <material>Gazebo/SkyBlue</material>
-  </gazebo>
-  <gazebo reference="arm_3_link">
-    <material>Gazebo/Yellow</material>
-  </gazebo>
-  <gazebo reference="arm_4_link">
-    <material>Gazebo/SkyBlue</material>
-  </gazebo>
-  <gazebo reference="arm_5_link">
-    <material>Gazebo/Yellow</material>
-  </gazebo>
   <!-- left sdh hand -->
-  <xacro:schunk_sdh name="left_hand" parent="arm_6_link">
-    <origin xyz="0 0 0.08"  rpy= "0 0 ${M_PI}"/>
-  </xacro:schunk_sdh>
-  <!-- right arm -->
-  <xacro:schunk_lwa4p name="right_arm" parent="body" has_podest="true">
-    <!--<origin xyz="0 0.18 0.08" rpy="1.5707 0 3.1415" />-->
-    <origin xyz="0.21 -0.24 0.42" rpy="${M_PI/2} 0 0" />
-  </xacro:schunk_lwa4p>
-  <gazebo reference="right_arm_1_link">
-    <material>Gazebo/Yellow</material>
-  </gazebo>
-  <gazebo reference="right_arm_2_link">
-    <material>Gazebo/SkyBlue</material>
-  </gazebo>
-  <gazebo reference="right_arm_3_link">
-    <material>Gazebo/Yellow</material>
-  </gazebo>
-  <gazebo reference="right_arm_4_link">
-    <material>Gazebo/SkyBlue</material>
-  </gazebo>
-  <gazebo reference="right_arm_5_link">
-    <material>Gazebo/Yellow</material>
-  </gazebo>
-  <!-- right sdh hand -->
-  <xacro:schunk_sdh name="right_hand" parent="right_arm_6_link">
+  <xacro:schunk_sdh name="left_hand" parent="left_arm_6_link">
     <origin xyz="0 0 0.08"  rpy= "0 0 0"/>
   </xacro:schunk_sdh>
-  <!-- ridgeback -->
-  <xacro:clearpath_ridgeback name="ridgeback">
-    <origin xyz="0 0 0" rpy="0 0 0" />
-  </xacro:clearpath_ridgeback>
-  <!-- backlift -->
-  <link name="backlift">
-    <collision>
-      <geometry>
-        <box size="0.1 0.4 0.8" />
-      </geometry>
-      <origin xyz="0 0 0.3" rpy="0 0 0" />
-    </collision>
-    <visual>
-      <geometry>
-        <box size="0.1 0.4 0.8" />
-        <!-- Backlift mesh available but box with prismatic joint may be more useful -->
-        <!--
-        <mesh filename="package://grasping_sim/urdf/meshes/humanoid/backliftlowres.stl" scale="0.001 0.001 0.001" />
-        -->
-      </geometry>
-      <origin xyz="0 0 0.3" rpy="0 0 0" />
-      <!-- Origin if using backlift mesh -->
-      <!-- <origin xyz="0.3 0.75 -0.3" rpy="${M_PI/2} 0 -${M_PI/2}" /> -->
-    </visual>
-    <inertial>
-      <origin xyz="0 0 0" rpy="0 0 0" />
-      <mass value="1" />
-      <inertia
-              ixx="1.0" ixy="0.0" ixz="0.0"
-              iyy="1.0" iyz="0.0"
-              izz="1.0" />
-    </inertial>
-  </link>
-  <gazebo reference="backlift">
-    <material>Gazebo/DarkGrey</material>
-  </gazebo>
-  <joint name="ridgeback_backlift" type="fixed">
-    <parent link="ridgeback_top_link" />
-    <child link="backlift" />
-    <origin xyz="0 0 ${deck_height}" rpy="0 0 0" />
+   <!-- right arm -->
+   <xacro:schunk_lwa4p name="right_arm" parent="body" has_podest="true">
+     <origin xyz="0 0.18 0.08" rpy="1.5707 0 3.1415" />
+   </xacro:schunk_lwa4p>
+   <!-- right sdh gripper -->
+   <xacro:schunk_sdh name="right_hand" parent="right_arm_6_link">
+    <origin xyz="0 0 0.08"  rpy= "0 0 3.1415"/>
+   </xacro:schunk_sdh>
+  <joint name="base_joint" type="fixed">
+    <parent link="world"/>
+    <child link="body"/>
   </joint>
-  <joint name="backlift_body" type="prismatic">
-    <parent link="backlift" />
-    <child link="body" />
-    <!-- Origin for box model of body -->
-    <!--<origin xyz="0.25 0 0.6" rpy="0 0 0" />-->
-    <!-- Origin for mesh model of body -->
-    <axis xyz="0 0 1" />
-    <limit effort="100.0" lower="-0.4" upper="0.1" velocity="0.1" />
-    <origin xyz="0 0 0.5" rpy="0 0 0" />
-  </joint>
-  <!-- Backlift and body transmission -->
-  <transmission name="backlift_body_trans">
-    <type>transmission_interface/SimpleTransmission</type>
-    <joint name="backlift_body">
-      <hardwareInterface>hardware_interface/PositionJointInterface</hardwareInterface>
-    </joint>
-    <actuator name="backlift_motor">
-      <mechanicalReduction>1</mechanicalReduction>
-    </actuator>
-  </transmission>
   <joint name="camera_joint" type="fixed">
     <parent link="head"/>
     <child link="zed_base_link"/>
-    <!-- <origin xyz=".155 0.03 1.14" rpy="0 0 -1.5707" /> -->
-    <origin xyz="0.0 0.0 0.0" rpy="0 0 0" />
+    <origin xyz=".155 0.03 1.14" rpy="0 0 -1.5707" />
   </joint>
   <!-- base_link -->
@@ -202,8 +84,7 @@
     <origin xyz="0 0 0" rpy="0 0 0" />
   </joint>
-  <link name="zed_camera_center"> <!-- Commented out to allow multiple cameras to see out head visor. -->
-  <!--
+  <link name="zed_camera_center">
     <visual>
-      <origin xyz="0.17 -0.005 0.09" rpy="0 0 0"/>
+      <origin xyz="0 0 0" rpy="0 0 0"/>
       <geometry>
         <mesh filename="package://grasping_sim/urdf/urdf/zed/models/ZED.stl" />
@@ -213,5 +94,4 @@
       </material>
     </visual>
-    -->
   </link>
   <!-- Left Camera -->
@@ -219,14 +99,14 @@
     <parent link="zed_camera_center"/>
     <child link="zed_left_camera_frame"/>
-    <origin xyz="0 0.0 0" rpy="0 0 0" />
+    <origin xyz="0 0.06 0" rpy="0 0 0" />
   </joint>
   <link name="zed_left_camera_frame" />
   <joint name="zed_left_camera_depth_joint" type="fixed">
-    <origin xyz="0.0 0.0 0.0" rpy="0 0 0"/>
+    <origin xyz="0.05 0.05 0.05" rpy="-1.5707 1.5707 -1.5707"/>
     <parent link="zed_left_camera_frame"/>
     <child link="zed_depth_frame"/>
   </joint>
   <joint name="zed_left_camera_optical_joint" type="fixed">
-    <origin xyz="0 0 0.0" rpy="0 0.0 0"/>
+    <origin xyz="0 0 0" rpy="-1.57079632679 0.0 -1.57079632679"/>
     <parent link="zed_left_camera_frame"/>
     <child link="zed_left_camera_optical_frame"/>
@@ -251,5 +131,5 @@
       <update_rate>15.0</update_rate>
       <camera name="head">
-        <pose>0.175 0 0.089 0 0 0.0</pose>
+        <pose>0.005 0 0 0 0 0</pose>
         <horizontal_fov>1.3962634</horizontal_fov>
         <image>
@@ -283,10 +163,9 @@
     </sensor>
   </gazebo>
-  <!-- depth camera -->
+<!-- depth camera -->
   <!-- Kamera -->
   <xacro:include filename="$(find luh_youbot_description)/urdf/sensors/asus_xtion_camera.urdf.xacro" />
   <xacro:asus_xtion_camera name="camera" parent="zed_depth_frame" tilt="0.0">
-    <!-- <origin xyz="0.08 -0.04 -0.05" rpy="0 -1.5707 0" /> -->
-    <origin xyz="0.16 -0.01 0.053" rpy="0 0 0" /> <!-- Same position as ZED camera -->
+    <origin xyz="0.08 -0.04 -0.05" rpy="0 -1.5707 0" />
   </xacro:asus_xtion_camera>
 <!-- ros_control plugin -->
@@ -296,6 +175,6 @@
 <!--  </gazebo>-->
   <gazebo>
-    <plugin name="ros_control" filename="libhwi_switch_gazebo_ros_control.so">
-    <robotNamespace></robotNamespace>
+    <plugin name="gazebo_ros_control" filename="libgazebo_ros_control.so">
+      <robotNamespace></robotNamespace>
     </plugin>
   </gazebo>
