Commit message: Added launch file for stationary humanoid with two arms. TF tree needs to be corrected.

File: simulation/grasping_sim/urdf/two_arm_robot.urdf.xacro (robot description, xacro)
@@ -39,4 +39,8 @@
       </geometry>
     </visual>
+    <inertial>
+      <mass value="10"/>
+      <inertia ixx="0.4" ixy="0.0" ixz="0.0" iyy="0.4" iyz="0.0" izz="0.2"/>
+    </inertial>
   </link>
   <gazebo reference="body">
@@ -56,4 +60,12 @@
       <origin xyz="0.2 -0.16 -1.05" rpy="0 0 ${M_PI/2}"/>
     </visual>
+    <inertial>
+        <origin xyz="0 0 0" rpy="0 0 0" />
+        <mass value="1" />
+        <inertia
+          ixx="1.0" ixy="0.0" ixz="0.0"
+          iyy="1.0" iyz="0.0"
+          izz="1.0" />
+    </inertial>
   </link>
   <gazebo reference="head">
