Commit message: Fixed collision shapes for head and body.

File: simulation/grasping_sim/urdf/full_robot.urdf.xacro (robot description, xacro)
@@ -21,5 +21,5 @@
 <!--      </geometry>-->
       <!--<origin xyz="-0.03 -.046 -0.038" rpy="0 0 0"/>-->
-      <origin xyz="0 0 0" rpy="0 0 0"/>
+      <origin xyz="0.27 0 0.28" rpy="0 0 0"/>
       <geometry>
         <box size="0.4 0.525 0.576" />
@@ -46,6 +46,8 @@
     <origin xyz="0 0 0" rpy="0 0 0"/>
     <collision>
-      <geometry>
-        <mesh filename="package://grasping_sim/urdf/meshes/humanoid/headconvexhull.stl" scale="0.001 0.001 0.001"/>
+      <origin xyz="0 0 0.1" rpy="0 0 0"/>
+      <geometry>
+        <!-- <mesh filename="package://grasping_sim/urdf/meshes/humanoid/headconvexhull.stl" scale="0.001 0.001 0.001"/> -->
+        <cylinder length="0.3" radius="0.19" />
       </geometry>
     </collision>

File: simulation/grasping_sim/urdf/two_arm_robot.urdf.xacro (robot description, xacro)
@@ -21,5 +21,5 @@
 <!--      </geometry>-->
       <!--<origin xyz="-0.03 -.046 -0.038" rpy="0 0 0"/>-->
-      <origin xyz="0 0 0" rpy="0 0 0"/>
+      <origin xyz="0.27 0 0.28" rpy="0 0 0"/>
       <geometry>
         <box size="0.4 0.525 0.576" />
@@ -50,6 +50,8 @@
     <origin xyz="0 0 0" rpy="0 0 0"/>
     <collision>
-      <geometry>
-        <mesh filename="package://grasping_sim/urdf/meshes/humanoid/headconvexhull.stl" scale="0.001 0.001 0.001"/>
+      <origin xyz="0 0 0.1" rpy="0 0 0"/>
+      <geometry>
+        <!-- <mesh filename="package://grasping_sim/urdf/meshes/humanoid/headconvexhull.stl" scale="0.001 0.001 0.001"/> -->
+        <cylinder length="0.3" radius="0.19" />
       </geometry>
     </collision>
